File: Bike logger/pcb/current_voltage_sensor/current_voltage_sensor.sch (KiCad schematic (older format))
At the start: 0 parts

Commit message: put together draft one of current voltage module
Parts:
- added J1: Conn_01x04, Connector:NS-Tech_Grove_1x04_P2mm_Vertical, symbol Connector_Generic:Conn_01x04
- added J2, J3: Conn_01x01, TerminalBlock_TE-Connectivity:TerminalBlock_TE_282834-2_1x02_P2.54mm_Horizontal, symbol Connector_Generic:Conn_01x01
- added JP1, JP2: SolderJumper_3_Open, Jumper:SolderJumper-3_P2.0mm_Open_TrianglePad1.0x1.5mm_NumberLabels, symbol Jumper:SolderJumper_3_Open
- added R1: 0.02 ohm, Resistor_SMD:R_Shunt_Ohmite_LVK25, symbol Device:R
- added R2, R3: 2K, Resistor_SMD:R_0402_1005Metric, symbol Device:R
- added TP1, TP2: TestPoint, TestPoint:TestPoint_Loop_D2.54mm_Drill1.5mm_Beaded, symbol Connector:TestPoint
- added U1: LTC4151, Package_DFN_QFN:DFN-10-1EP_3x3mm_P0.5mm_EP1.55x2.48mm, symbol custom_symbols:LTC4151
Connections:
- new net: TP2.1, U1.5 (ADIN)
- new net: TP1.1, U1.8 (#SHDN)
- new net +3V3: J1.3 (Pin_3), R2.1, R3.1
- new net ADR0: JP1.2 (C), U1.4 (ADR0)
- new net ADR1: JP2.2 (C), U1.3 (ADR1)
- new net GND: J1.4 (Pin_4), JP1.3 (B), JP2.3 (B), U1.9 (GND)
- new net SCL: J1.1 (Pin_1), R3.2, U1.6 (SCL)
- new net SDA: J1.2 (Pin_2), R2.2, U1.7 (SDA)
- new net SENSE+: J3.1 (Pin_1), JP1.1 (A), JP2.1 (A), R1.2, U1.1 (SENSE+), U1.2 (Vin)
- new net SENSE-: J2.1 (Pin_1), R1.1, U1.10 (SENSE-)

Commit message: update footprints
Parts:
- TP1, TP2: footprint TestPoint:TestPoint_Loop_D2.54mm_Drill1.5mm_Beaded -> TestPoint:TestPoint_THTPad_D2.0mm_Drill1.0mm
- U1: min_qty (none) -> 1; price (none) -> 1.96; purchase_link (none) -> https://uk.farnell.com/linear-technology/ltc4151cdd-pbf/mon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
Changed lines of the file:
@@
 EESchema Schematic File Version 4
+LIBS:current_voltage_sensor-cache
 EELAYER 29 0
 EELAYER END
@@
 F 0 "TP1" V 7154 3738 50  0000 L CNN
 F 1 "TestPoint" V 7245 3738 50  0000 L CNN
-F 2 "TestPoint:TestPoint_Loop_D2.54mm_Drill1.5mm_Beaded" H 7400 3550 50  0001 C CNN
+F 2 "TestPoint:TestPoint_THTPad_D2.0mm_Drill1.0mm" H 7400 3550 50  0001 C CNN
 F 3 "~" H 7400 3550 50  0001 C CNN
 	1    7200 3550
@@
 F 0 "TP2" V 7154 3938 50  0000 L CNN
 F 1 "TestPoint" V 7245 3938 50  0000 L CNN
-F 2 "TestPoint:TestPoint_Loop_D2.54mm_Drill1.5mm_Beaded" H 7400 3750 50  0001 C CNN
+F 2 "TestPoint:TestPoint_THTPad_D2.0mm_Drill1.0mm" H 7400 3750 50  0001 C CNN
 F 3 "~" H 7400 3750 50  0001 C CNN
 	1    7200 3750
@@
 F 2 "Package_DFN_QFN:DFN-10-1EP_3x3mm_P0.5mm_EP1.55x2.48mm" H 5800 3250 50  0001 C CNN
 F 3 "" H 5800 3250 50  0001 C CNN
+F 4 "1" H 5900 3250 50  0001 C CNN "min_qty"
+F 5 "1.96" H 5900 3250 50  0001 C CNN "price"
+F 6 "https://uk.farnell.com/linear-technology/ltc4151cdd-pbf/monitor-current-voltage-i2c-10dfn/dp/2295457?scope=partnumberlookahead&ost=LTC4151CDD%23PBF&searchref=searchlookahead&exaMfpn=true" H 5900 3250 50  0001 C CNN "purchase_link"
 	1    5900 3250
 	1    0    0    -1

Commit message: organise diagram
Other:
- note added: "Connection to High current path to measure"
- note added: "Connection to mother board"
- note added: "I2C address selection"
- note added: "LTC4151 sensor IC"
- note added: "Shunt resistor section"
- moved on the sheet: J1, J2, J3, R1
Changed lines of the file:
@@
 L Connector_Generic:Conn_01x04 J1
 U 1 1 6015676D
-P 8600 3550
-F 0 "J1" H 8680 3542 50  0000 L CNN
-F 1 "Conn_01x04" H 8680 3451 50  0000 L CNN
-F 2 "Connector:NS-Tech_Grove_1x04_P2mm_Vertical" H 8600 3550 50  0001 C CNN
-F 3 "~" H 8600 3550 50  0001 C CNN
-	1    8600 3550
+P 9450 2800
+F 0 "J1" H 9530 2792 50  0000 L CNN
+F 1 "Conn_01x04" H 9530 2701 50  0000 L CNN
+F 2 "Connector:NS-Tech_Grove_1x04_P2mm_Vertical" H 9450 2800 50  0001 C CNN
+F 3 "~" H 9450 2800 50  0001 C CNN
+	1    9450 2800
 	1    0    0    -1
 $EndComp
@@
 Text Label 7100 3450 2    50   ~ 0
 SDA
-Text Label 8150 3450 0    50   ~ 0
+Text Label 9000 2700 0    50   ~ 0
 SCL
 Wire Wire Line
-	8400 3450 8150 3450
-Text Label 8150 3550 0    50   ~ 0
+	9250 2700 9000 2700
+Text Label 9000 2800 0    50   ~ 0
 SDA
 Wire Wire Line
-	8400 3550 8150 3550
-Wire Wire Line
-	8400 3750 8300 3750
-Wire Wire Line
-	8300 3750 8300 3850
+	9250 2800 9000 2800
+Wire Wire Line
+	9250 3000 9150 3000
+Wire Wire Line
+	9150 3000 9150 3100
 $Comp
 L power:GND #PWR05
 U 1 1 6015C57C
-P 8300 3850
-F 0 "#PWR05" H 8300 3600 50  0001 C CNN
-F 1 "GND" H 8305 3677 50  0000 C CNN
-F 2 "" H 8300 3850 50  0001 C CNN
-F 3 "" H 8300 3850 50  0001 C CNN
-	1    8300 3850
+P 9150 3100
+F 0 "#PWR05" H 9150 2850 50  0001 C CNN
+F 1 "GND" H 9155 2927 50  0000 C CNN
+F 2 "" H 9150 3100 50  0001 C CNN
+F 3 "" H 9150 3100 50  0001 C CNN
+	1    9150 3100
 	1    0    0    -1
 $EndComp
@@
 	6650 3650 6650 4100
 Wire Wire Line
-	8400 3650 7950 3650
-Wire Wire Line
-	7950 3650 7950 3600
+	9250 2900 8800 2900
+Wire Wire Line
+	8800 2900 8800 2850
 $Comp
 L power:+3.3V #PWR04
 U 1 1 6015E541
-P 7950 3600
-F 0 "#PWR04" H 7950 3450 50  0001 C CNN
-F 1 "+3.3V" H 7965 3773 50  0000 C CNN
-F 2 "" H 7950 3600 50  0001 C CNN
-F 3 "" H 7950 3600 50  0001 C CNN
-	1    7950 3600
+P 8800 2850
+F 0 "#PWR04" H 8800 2700 50  0001 C CNN
+F 1 "+3.3V" H 8815 3023 50  0000 C CNN
+F 2 "" H 8800 2850 50  0001 C CNN
+F 3 "" H 8800 2850 50  0001 C CNN
+	1    8800 2850
 	1    0    0    -1
 $EndComp
@@
 L Device:R R1
 U 1 1 6016433A
-P 4650 2250
-F 0 "R1" V 4443 2250 50  0000 C CNN
-F 1 "0.02 ohm" V 4534 2250 50  0000 C CNN
-F 2 "Resistor_SMD:R_Shunt_Ohmite_LVK25" V 4580 2250 50  0001 C CNN
-F 3 "~" H 4650 2250 50  0001 C CNN
-	1    4650 2250
+P 3550 2250
+F 0 "R1" V 3343 2250 50  0000 C CNN
+F 1 "0.02 ohm" V 3434 2250 50  0000 C CNN
+F 2 "Resistor_SMD:R_Shunt_Ohmite_LVK25" V 3480 2250 50  0001 C CNN
+F 3 "~" H 3550 2250 50  0001 C CNN
+	1    3550 2250
 	0    1    1    0
 $EndComp
 Wire Wire Line
-	4500 2250 4300 2250
-Wire Wire Line
-	4800 2250 4950 2250
-Text Label 4300 2450 3    50   ~ 0
+	3400 2250 3200 2250
+Wire Wire Line
+	3700 2250 3850 2250
+Text Label 3200 2450 3    50   ~ 0
 SENSE+
 Wire Wire Line
-	4300 2250 4300 2450
-Connection ~ 4300 2250
-Wire Wire Line
-	4300 2250 3850 2250
-Text Label 4950 2450 3    50   ~ 0
+	3200 2250 3200 2450
+Connection ~ 3200 2250
+Wire Wire Line
+	3200 2250 2750 2250
+Text Label 3850 2450 3    50   ~ 0
 SENSE-
 Wire Wire Line
-	4950 2450 4950 2250
-Connection ~ 4950 2250
-Wire Wire Line
-	4950 2250 5300 2250
-Text Label 3850 2250 0    50   ~ 0
-Vin
-Text Label 5300 2250 2    50   ~ 0
+	3850 2450 3850 2250
+Connection ~ 3850 2250
+Wire Wire Line
+	3850 2250 4200 2250
+Text Label 2750 2250 0    50   ~ 0
+Vin
+Text Label 4200 2250 2    50   ~ 0
 Vout
 Text Label 5050 3450 0    50   ~ 0
@@
 L Connector_Generic:Conn_01x01 J2
 U 1 1 6018A246
-P 6700 4600
-F 0 "J2" H 6780 4642 50  0000 L CNN
-F 1 "Conn_01x01" H 6780 4551 50  0000 L CNN
-F 2 "TerminalBlock_TE-Connectivity:TerminalBlock_TE_282834-2_1x02_P2.54mm_Horizontal" H 6700 4600 50  0001 C CNN
-F 3 "~" H 6700 4600 50  0001 C CNN
-	1    6700 4600
+P 9200 4200
+F 0 "J2" H 9280 4242 50  0000 L CNN
+F 1 "Conn_01x01" H 9280 4151 50  0000 L CNN
+F 2 "TerminalBlock_TE-Connectivity:TerminalBlock_TE_282834-2_1x02_P2.54mm_Horizontal" H 9200 4200 50  0001 C CNN
+F 3 "~" H 9200 4200 50  0001 C CNN
+	1    9200 4200
 	1    0    0    -1
 $EndComp
@@
 L Connector_Generic:Conn_01x01 J3
 U 1 1 6018A9BE
-P 6700 4850
-F 0 "J3" H 6780 4892 50  0000 L CNN
-F 1 "Conn_01x01" H 6780 4801 50  0000 L CNN
-F 2 "TerminalBlock_TE-Connectivity:TerminalBlock_TE_282834-2_1x02_P2.54mm_Horizontal" H 6700 4850 50  0001 C CNN
-F 3 "~" H 6700 4850 50  0001 C CNN
-	1    6700 4850
-	1    0    0    -1
-$EndComp
-Text Label 6250 4600 0    50   ~ 0
+P 9200 4450
+F 0 "J3" H 9280 4492 50  0000 L CNN
+F 1 "Conn_01x01" H 9280 4401 50  0000 L CNN
+F 2 "TerminalBlock_TE-Connectivity:TerminalBlock_TE_282834-2_1x02_P2.54mm_Horizontal" H 9200 4450 50  0001 C CNN
+F 3 "~" H 9200 4450 50  0001 C CNN
+	1    9200 4450
+	1    0    0    -1
+$EndComp
+Text Label 8750 4200 0    50   ~ 0
 Vout
-Text Label 6250 4850 0    50   ~ 0
-Vin
-Wire Wire Line
-	6250 4850 6500 4850
-Wire Wire Line
-	6500 4600 6250 4600
+Text Label 8750 4450 0    50   ~ 0
+Vin
+Wire Wire Line
+	8750 4450 9000 4450
+Wire Wire Line
+	9000 4200 8750 4200
 $Comp
 L Jumper:SolderJumper_3_Open JP2
@@
 Text Label 3350 4750 3    50   ~ 0
 ADR0
+Wire Notes Line
+	2350 3100 4500 3100
+Wire Notes Line
+	4500 3100 4500 5350
+Wire Notes Line
+	4500 5350 2350 5350
+Wire Notes Line
+	2350 5350 2350 3100
+Text Notes 2450 3200 0    50   ~ 0
+I2C address selection
+Text Notes 2650 1800 0    50   ~ 0
+Shunt resistor section
+Wire Notes Line
+	2450 1650 2450 2900
+Wire Notes Line
+	2450 2900 4450 2900
+Wire Notes Line
+	4450 2900 4450 1650
+Wire Notes Line
+	4450 1650 2450 1650
+Wire Notes Line
+	8450 5000 10350 5000
+Wire Notes Line
+	10350 5000 10350 2350
+Wire Notes Line
+	10350 2350 8450 2350
+Wire Notes Line
+	8450 3600 10350 3600
+Wire Notes Line
+	8450 2350 8450 5000
+Text Notes 8600 2500 0    50   ~ 0
+Connection to mother board
+Text Notes 8550 3800 0    50   ~ 0
+Connection to High current path to measure
+Text Notes 5150 2250 0    50   ~ 0
+LTC4151 sensor IC
+Wire Notes Line
+	4750 1900 4750 4900
+Wire Notes Line
+	4750 4900 7900 4900
+Wire Notes Line
+	7900 4900 7900 1900
+Wire Notes Line
+	7900 1900 4750 1900
 $EndSCHEMATC

Commit message: Update current_voltage_sensor.sch
Parts:
- added TP3, TP4, TP5, TP6: TestPoint, TestPoint:TestPoint_THTPad_D2.0mm_Drill1.0mm, symbol Connector:TestPoint
- added U?: INA226, Package_SO:MSOP-10_3x3mm_P0.5mm, symbol Analog_ADC:INA226
Connections:
- net SCL: now also TP3.1
- net SDA: now also TP4.1
- net SENSE+: now also TP5.1
- net SENSE-: now also TP6.1
Other:
- note added: "I2C pullups"
- note added: "Test points to verify voltage drop"
